Commit message: Update mobile robot swerve descriptions

File: src/mobile_robot/description_mobile/urdf/mech/virtual_swerve_module.urdf.xacro (robot description, xacro)
@@ -1,155 +1,85 @@
 <?xml version="1.0"?>
 <robot xmlns:xacro="http://ros.org/wiki/xacro">
-    <xacro:macro name="virtual_swerve_module" params="
+  <xacro:macro name="virtual_swerve_module" params="
         prefix parent
         pos_x pos_y pos_z"
     >
-  <!-- virtual rear  left steering -->
+    <!--********************************************* STEERING *****************************************************************   -->
+    <!-- virtual front right steering -->
+    <link name="${prefix}virtual_front_right_steering_link">
+    </link>
+    <joint name="${prefix}virtual_front_right_steering_joint" type="revolute">
+      <parent link="${parent}"/>
+      <child link="${prefix}virtual_front_right_steering_link"/>
+      <origin xyz="${pos_x} -${pos_y} ${pos_z}" rpy="0 0 0"/>
+      <axis xyz="0 0 1"/>
+      <limit lower="-3.14159" upper="3.14159" effort="100.0" velocity="10.0"/>
+    </joint>
+    <!-- virtual rear left steering -->
     <link name="${prefix}virtual_rear_left_steering_link">
-      <visual>
-        <origin xyz="0 0 0" rpy="0 0 0"/>
-        <geometry>
-           <cylinder length="${rulment_axial_height}" radius="${rulment_axial_diametru}"/>
-        </geometry>
-        <material name="invisible"/>
-      </visual>
     </link>
     <joint name="${prefix}virtual_rear_left_steering_joint" type="revolute">
-      <parent link="${prefix}${parent}"/>
+      <parent link="${parent}"/>
       <child link="${prefix}virtual_rear_left_steering_link"/>
-      <origin xyz="-${pos_x} ${pos_y} -${pos_z}" rpy="0 0 0"/>
+      <origin xyz="-${pos_x} ${pos_y} ${pos_z}" rpy="0 0 0"/>
       <axis xyz="0 0 1"/>
-      <limit lower="-1.0" upper="1.0" effort="100.0" velocity="0.0"/>
-      <dynamics damping="0.2"/>
+      <limit lower="-3.14159" upper="3.14159" effort="100.0" velocity="10.0"/>
     </joint>
     <!-- virtual rear right steering -->
     <link name="${prefix}virtual_rear_right_steering_link">
-      <visual>
-        <origin xyz="0 0 0" rpy="0 0 0"/>
-        <geometry>
-          <cylinder length="${rulment_axial_height}" radius="${rulment_axial_diametru}"/>
-        </geometry>
-        <material name="invisible"/>
-      </visual>
     </link>
     <joint name="${prefix}virtual_rear_right_steering_joint" type="revolute">
-      <parent link="${prefix}${parent}"/>
+      <parent link="${parent}"/>
       <child link="${prefix}virtual_rear_right_steering_link"/>
-      <origin xyz="-${pos_x} -${pos_y} -${pos_z}" rpy="0 0 0"/>
+      <origin xyz="-${pos_x} -${pos_y} ${pos_z}" rpy="0 0 0"/>
       <axis xyz="0 0 1"/>
-      <limit lower="-1.0" upper="1.0" effort="100.0" velocity="0.0"/>
-      <dynamics damping="0.2"/>
-      <!-- <mimic joint="${prefix}virtual_front_right_steering_joint" multiplier="1.0" offset="0.0"/> -->
+      <limit lower="-3.14159" upper="3.14159" effort="100.0" velocity="10.0"/>
     </joint>
-   <!-- virtual front left steering -->
+    <!-- virtual front left steering -->
     <link name="${prefix}virtual_front_left_steering_link">
-      <visual>
-        <origin xyz="0 0 0" rpy="0 0 0"/>
-        <geometry>
-          <cylinder length="${rulment_axial_height}" radius="${rulment_axial_diametru}"/>
-        </geometry>
-        <material name="invisible"/>
-      </visual>
     </link>
     <joint name="${prefix}virtual_front_left_steering_joint" type="revolute">
-      <parent link="${prefix}${parent}"/>
+      <parent link="${parent}"/>
       <child link="${prefix}virtual_front_left_steering_link"/>
-      <origin xyz="${pos_x} ${pos_y} -${pos_z}" rpy="0 0 0"/>
+      <origin xyz="${pos_x} ${pos_y} ${pos_z}" rpy="0 0 0"/>
       <axis xyz="0 0 1"/>
-      <limit lower="-1.0" upper="1.0" effort="100.0" velocity="0.0"/>
-      <dynamics damping="0.2"/>
-      <!-- <mimic joint="${prefix}virtual_rear_left_steering_joint" multiplier="1.0" offset="0.0"/> -->
+      <limit lower="-3.14159" upper="3.14159" effort="100.0" velocity="10.0"/>
     </joint>
-   <!-- virtual front right steering -->
-    <link name="${prefix}virtual_front_right_steering_link">
-      <visual>
-        <origin xyz="0 0 0" rpy="0 0 0"/>
-        <geometry>
-          <cylinder length="0.01" radius="${wheel_radius}"/>
-        </geometry>
-        <material name="invisible"/>
-      </visual>
+    <!--********************************************* TRACTION *****************************************************************   -->
+    <!-- virtual front right wheel -->
+    <link name="${prefix}virtual_front_right_wheel_link">
     </link>
-    <joint name="${prefix}virtual_front_right_steering_joint" type="revolute">
-      <parent link="${prefix}${parent}"/>
-      <child link="${prefix}virtual_front_right_steering_link"/>
-      <origin xyz="${pos_x} -${pos_y} -${pos_z}" rpy="0 0 0"/>
-      <axis xyz="0 0 1"/>
-      <limit lower="-1.0" upper="1.0" effort="100.0" velocity="0.0"/>
-      <dynamics damping="0.2"/>
+    <joint name="${prefix}virtual_front_right_wheel_joint" type="continuous">
+      <parent link="${prefix}virtual_front_right_steering_link"/>
+      <child link="${prefix}virtual_front_right_wheel_link"/>
+      <origin xyz="0 0 0" rpy="0 0 0"/>
+      <axis xyz="0 1 0"/>
     </joint>
-  <!-- virtual rear  left wheel -->
+    <!-- virtual rear left wheel RL -->
     <link name="${prefix}virtual_rear_left_wheel_link">
-      <visual>
-        <origin xyz="0 0 0" rpy="${PI/2} 0 ${PI/2}"/>
-        <geometry>
-          <cylinder length="0.01" radius="${wheel_radius}"/>
-        </geometry>
-        <material name="invisible"/>
-      </visual>
     </link>
     <joint name="${prefix}virtual_rear_left_wheel_joint" type="continuous">
-      <parent link="${prefix}virtual_rear_left_steering_link" />
-      <child link="${prefix}virtual_rear_left_wheel_link" />
-      <origin xyz="0 0 -${rulment_axial_height/2 + wheel_radius}" rpy="0 0 0"/>
-      <axis xyz="1 0 0"/>
-      <limit effort="100.0" velocity="100.0"/>
-      <dynamics damping="0.2"/>
+      <parent link="${prefix}virtual_rear_left_steering_link"/>
+      <child link="${prefix}virtual_rear_left_wheel_link"/>
+      <origin xyz="0 0 0" rpy="0 0 0"/>
+      <axis xyz="0 1 0"/>
     </joint>
-    <!-- virtual rear right wheel -->
+    <!-- virtual rear right wheel RR -->
     <link name="${prefix}virtual_rear_right_wheel_link">
-      <visual>
-        <origin xyz="0 0 0" rpy="${PI/2} 0 ${PI/2}"/>
-        <geometry>
-          <cylinder length="0.01" radius="${wheel_radius}"/>
-        </geometry>
-        <material name="invisible"/>
-      </visual>
     </link>
     <joint name="${prefix}virtual_rear_right_wheel_joint" type="continuous">
       <parent link="${prefix}virtual_rear_right_steering_link"/>
       <child link="${prefix}virtual_rear_right_wheel_link"/>
-      <origin xyz="0 0 -${rulment_axial_height/2 + wheel_radius}" rpy="0 0 0"/>
-      <axis xyz="1 0 0"/>
-      <limit effort="100.0" velocity="100.0"/>
-      <dynamics damping="0.2"/>
-      <!--<mimic joint="${prefix}virtual_front_right_wheel_joint" multiplier="1.0" offset="0.0"/> -->
+      <origin xyz="0 0 0" rpy="0 0 0"/>
+      <axis xyz="0 1 0"/>
     </joint>
-   <!-- virtual front left wheel -->
+    <!-- virtual front left wheel -->
     <link name="${prefix}virtual_front_left_wheel_link">
-      <visual>
-        <origin xyz="0 0 0" rpy="${PI/2} 0 ${PI/2}"/>
-        <geometry>
-          <cylinder length="0.01" radius="${wheel_radius}"/>
-        </geometry>
-        <material name="invisible"/>
-      </visual>
     </link>
     <joint name="${prefix}virtual_front_left_wheel_joint" type="continuous">
-      <parent link="${prefix}virtual_front_left_steering_link" />
-      <child link="${prefix}virtual_front_left_wheel_link" />
-      <origin xyz="0 0 -${rulment_axial_height/2 + wheel_radius}" rpy="0 0 0"/>
-      <axis xyz="1 0 0"/>
-      <limit effort="100.0" velocity="100.0"/>
-      <dynamics damping="0.2"/>
-      <!-- <mimic joint="${prefix}virtual_rear_left_wheel_joint" multiplier="1.0" offset="0.0"/> -->
-    </joint>
-   <!-- virtual front right wheel -->
-    <link name="${prefix}virtual_front_right_wheel">
-      <visual>
-        <origin xyz="0 0 0" rpy="${PI/2} 0 ${PI/2}"/>
-        <geometry>
-          <cylinder length="0.01" radius="${wheel_radius}"/>
-        </geometry>
-        <material name="invisible"/>
-      </visual>
-    </link>
-    <joint name="${prefix}virtual_front_right_wheel_joint" type="continuous">
-      <parent link="${prefix}virtual_front_right_steering_link"/>
-      <child link="${prefix}virtual_front_right_wheel"/>
-      <origin xyz="0 0 -${rulment_axial_height/2 + wheel_radius}" rpy="0 0 0"/>
-      <axis xyz="1 0 0"/>
-      <limit effort="100.0" velocity="100.0"/>
-      <dynamics damping="0.2"/>
+      <parent link="${prefix}virtual_front_left_steering_link"/>
+      <child link="${prefix}virtual_front_left_wheel_link"/>
+      <origin xyz="0 0 0" rpy="0 0 0"/>
+      <axis xyz="0 1 0"/>
     </joint>
   </xacro:macro>

File: src/mobile_robot/description_mobile/urdf/robots/swerveBOT_510.urdf.xacro (robot description, xacro)
@@ -4,5 +4,5 @@
   <xacro:arg name="name" default="amr"/>
   <!-- import main macro -->
-  <xacro:include filename="$(find description_mobile)/urdf/robots/swerveBOT_910_macro.xacro"/>
+  <xacro:include filename="$(find description_mobile)/urdf/robots/swerveBOT_510_macro.xacro"/>
   <!-- parameters -->
   <xacro:arg name="namespace" default="" />
@@ -32,5 +32,5 @@
       component_name="front_lidar"
       model="a2m8"
-      xyz="${str(base_length/2 - 0.045)} -${str(base_width/2 - 0.045)} -0.075"
+      xyz="${str(base_length/2 - 0.0)} -${str(base_width/2 - 0.0)} -0.0"
       rpy="0.0 0.0 -0.785398"
   />
@@ -40,5 +40,5 @@
       component_name="back_lidar"
       model="a2m8"
-      xyz="-${str(base_length/2 - 0.045)} ${str(base_width/2 - 0.045)} -0.062"
+      xyz="-${str(base_length/2 - 0.0)} ${str(base_width/2 - 0.0)} -0.0"
       rpy="0.0 0.0 2.356194"
   />

File: src/mobile_robot/description_mobile/urdf/robots/swerveBOT_510_macro.xacro (robot description, xacro)
@@ -4,5 +4,5 @@
     <!-- import main macro -->
     <xacro:include filename="$(find description_mobile)/meshes/materials.xacro" />
-    <xacro:include filename="$(find description_mobile)/urdf/properties/properties_swerveBOT_910.urdf.xacro"/>
+    <xacro:include filename="$(find description_mobile)/urdf/properties/properties_swerveBOT_510.urdf.xacro"/>
     <xacro:include filename="$(find description_mobile)/urdf/mech/chassis.urdf.xacro"/>
     <xacro:include filename="$(find description_mobile)/urdf/mech/diff_drive_module.urdf.xacro"/>
@@ -58,5 +58,5 @@
             steering_pos="virtual_rear_left"
         >
-        <origin xyz="-${wheelbase/2} ${wheel_track/2} -${base_height/2 + rulment_axial_height/2}" rpy="0 0 0"/>
+        <origin xyz="-${wheelbase/2} ${wheel_track/2} -${base_height/2 + rulment_axial_height/2}" rpy="0 0 3.14"/>
         </xacro:diff_drive_module>
         <xacro:diff_drive_module
@@ -68,5 +68,5 @@
             steering_pos="virtual_rear_right"
         >
-        <origin xyz="-${wheelbase/2} -${wheel_track/2} -${base_height/2 + rulment_axial_height/2}" rpy="0 0 0"/>
+        <origin xyz="-${wheelbase/2} -${wheel_track/2} -${base_height/2 + rulment_axial_height/2}" rpy="0 0 3.14"/>
         </xacro:diff_drive_module>
         <!-- ros2_control -->

File: src/mobile_robot/description_mobile/urdf/robots/swerve_2BOT_510.urdf.xacro (robot description, xacro)
@@ -4,5 +4,5 @@
   <xacro:arg name="name" default="amr"/>
   <!-- import main macro -->
-  <xacro:include filename="$(find description_mobile)/urdf/robots/swerveBOT_910_macro.xacro"/>
+  <xacro:include filename="$(find description_mobile)/urdf/robots/swerve_2BOT_510_macro.xacro"/>
   <!-- parameters -->
   <xacro:arg name="namespace" default="" />
@@ -26,5 +26,5 @@
       xyz="${str(base_length/2)} 0 -0.037"
       rpy="0.0 0.0 0.0"
-  /> -->
+  />
   <xacro:lidar.slamtec_rplidar
       parent_link="chassis_link"
@@ -32,5 +32,5 @@
       component_name="front_lidar"
       model="a2m8"
-      xyz="${str(base_length/2 - 0.045)} -${str(base_width/2 - 0.045)} -0.075"
+      xyz="${str(base_length/2 - 0.0)} -${str(base_width/2 - 0.0)} -0.0"
       rpy="0.0 0.0 -0.785398"
   />
@@ -40,6 +40,7 @@
       component_name="back_lidar"
       model="a2m8"
-      xyz="-${str(base_length/2 - 0.045)} ${str(base_width/2 - 0.045)} -0.062"
+      xyz="-${str(base_length/2 - 0.0)} ${str(base_width/2 - 0.0)} -0.0"
       rpy="0.0 0.0 2.356194"
   />
+  -->
 </robot>

File: src/mobile_robot/description_mobile/urdf/robots/swerve_2BOT_510_macro.xacro (robot description, xacro)
@@ -4,10 +4,10 @@
     <!-- import main macro -->
     <xacro:include filename="$(find description_mobile)/meshes/materials.xacro" />
-    <xacro:include filename="$(find description_mobile)/urdf/properties/properties_swerveBOT_910.urdf.xacro"/>
+    <xacro:include filename="$(find description_mobile)/urdf/properties/properties_swerveBOT_510.urdf.xacro"/>
     <xacro:include filename="$(find description_mobile)/urdf/mech/chassis.urdf.xacro"/>
     <xacro:include filename="$(find description_mobile)/urdf/mech/diff_drive_module.urdf.xacro"/>
     <xacro:include filename="$(find description_mobile)/urdf/mech/virtual_swerve_module.urdf.xacro"/>
     <xacro:include filename="$(find description_mobile)/urdf/mech/rear_wheels.urdf.xacro"/>
-    <xacro:include filename="$(find description_mobile)/ros2_control/swerve.ros2_control.xacro" />
+    <xacro:include filename="$(find description_mobile)/ros2_control/swerve_2BOT.ros2_control.xacro" />
     <xacro:include filename="$(find description_mobile)/ros2_control/drive_module.ros2_control.xacro" />
     <xacro:macro name="mobile_robot" params= "
@@ -33,14 +33,4 @@
             namespace="$(arg namespace)"
             prefix="$(arg prefix)"
-            name="diffBOT_FL"
-            parent="chassis_link"
-            drive_pos="FL_"
-            steering_pos="virtual_front_left"
-        >
-        <origin xyz="${wheelbase/2} ${wheel_track/2} -${base_height/2 + rulment_axial_height/2}" rpy="0 0 0"/>
-        </xacro:diff_drive_module>
-        <xacro:diff_drive_module
-            namespace="$(arg namespace)"
-            prefix="$(arg prefix)"
             name="diffBOT_FR"
             parent="chassis_link"
@@ -58,15 +48,5 @@
             steering_pos="virtual_rear_left"
         >
-        <origin xyz="-${wheelbase/2} ${wheel_track/2} -${base_height/2 + rulment_axial_height/2}" rpy="0 0 0"/>
-        </xacro:diff_drive_module>
-        <xacro:diff_drive_module
-            namespace="$(arg namespace)"
-            prefix="$(arg prefix)"
-            name="diffBOT_RR"
-            parent="chassis_link"
-            drive_pos="RR_"
-            steering_pos="virtual_rear_right"
-        >
-        <origin xyz="-${wheelbase/2} -${wheel_track/2} -${base_height/2 + rulment_axial_height/2}" rpy="0 0 0"/>
+        <origin xyz="-${wheelbase/2} ${wheel_track/2} -${base_height/2 + rulment_axial_height/2}" rpy="0 0 3.14"/>
         </xacro:diff_drive_module>
         <!-- ros2_control -->

Commit message: Add Balena robot stack deployment

File: src/mobile_robot/description_mobile/urdf/mech/virtual_swerve_module.urdf.xacro (robot description, xacro)
@@ -14,5 +14,5 @@
       <origin xyz="${pos_x} -${pos_y} ${pos_z}" rpy="0 0 0"/>
       <axis xyz="0 0 1"/>
-      <limit lower="-3.14159" upper="3.14159" effort="100.0" velocity="10.0"/>
+      <limit lower="-${PI}" upper="${PI}" effort="100.0" velocity="10.0"/>
     </joint>
     <!-- virtual rear left steering -->
@@ -24,5 +24,5 @@
       <origin xyz="-${pos_x} ${pos_y} ${pos_z}" rpy="0 0 0"/>
       <axis xyz="0 0 1"/>
-      <limit lower="-3.14159" upper="3.14159" effort="100.0" velocity="10.0"/>
+      <limit lower="-${PI}" upper="${PI}" effort="100.0" velocity="10.0"/>
     </joint>
     <!-- virtual rear right steering -->
@@ -34,5 +34,5 @@
       <origin xyz="-${pos_x} -${pos_y} ${pos_z}" rpy="0 0 0"/>
       <axis xyz="0 0 1"/>
-      <limit lower="-3.14159" upper="3.14159" effort="100.0" velocity="10.0"/>
+      <limit lower="-${PI}" upper="${PI}" effort="100.0" velocity="10.0"/>
     </joint>
     <!-- virtual front left steering -->
@@ -44,5 +44,5 @@
       <origin xyz="${pos_x} ${pos_y} ${pos_z}" rpy="0 0 0"/>
       <axis xyz="0 0 1"/>
-      <limit lower="-3.14159" upper="3.14159" effort="100.0" velocity="10.0"/>
+      <limit lower="-${PI}" upper="${PI}" effort="100.0" velocity="10.0"/>
     </joint>
     <!--********************************************* TRACTION *****************************************************************   -->
