Commit message: Add fused odometry and stabilize swerve visualization

File: src/mobile_robot/description_mobile/ros2_control/wheelbot_serial_swerve_2bot.ros2_control.xacro (robot description, xacro)
@@ -2,5 +2,5 @@
 <robot xmlns:xacro="http://www.ros.org/wiki/xacro">
   <xacro:macro name="wheelbot_serial_swerve_2bot_ros2_control"
-    params="name prefix serial_port baudrate command_timeout_ms active_modules wheel_radius wheel_drive_len">
+    params="name prefix serial_port baudrate command_timeout_ms active_modules wheel_radius wheel_drive_len imu_topic imu_frame_id">
     <ros2_control name="${name}" type="system">
       <hardware>
@@ -10,8 +10,11 @@
         <param name="command_timeout_ms">${command_timeout_ms}</param>
         <param name="active_modules">${active_modules}</param>
+        <param name="imu_topic">${imu_topic}</param>
+        <param name="imu_frame_id">${imu_frame_id}</param>
         <param name="wheel_radius">${wheel_radius}</param>
         <param name="wheel_drive_len">${wheel_drive_len}</param>
-        <param name="steering_drive_mode">smooth_arc</param>
-        <param name="steering_alignment_tolerance">0.08</param>
+        <param name="steering_drive_mode">strict_gate</param>
+        <param name="steering_gain">0.35</param>
+        <param name="steering_alignment_tolerance">0.10</param>
         <param name="steering_min_speed_scale">0.15</param>
         <param name="steering_zero_speed_error">1.20</param>
@@ -67,4 +70,28 @@
         <state_interface name="velocity"/>
       </joint>
+      <joint name="${prefix}FR_drive_right_joint">
+        <state_interface name="position"/>
+        <state_interface name="velocity"/>
+      </joint>
+      <joint name="${prefix}FR_drive_left_joint">
+        <state_interface name="position"/>
+        <state_interface name="velocity"/>
+      </joint>
+      <joint name="${prefix}FR_steering_joint">
+        <state_interface name="position"/>
+        <state_interface name="velocity"/>
+      </joint>
+      <joint name="${prefix}RL_drive_right_joint">
+        <state_interface name="position"/>
+        <state_interface name="velocity"/>
+      </joint>
+      <joint name="${prefix}RL_drive_left_joint">
+        <state_interface name="position"/>
+        <state_interface name="velocity"/>
+      </joint>
+      <joint name="${prefix}RL_steering_joint">
+        <state_interface name="position"/>
+        <state_interface name="velocity"/>
+      </joint>
     </ros2_control>
   </xacro:macro>

File: src/mobile_robot/description_mobile/urdf/mech/serial_diff_drive_module.urdf.xacro (robot description, xacro)
@@ -24,7 +24,6 @@
       <child link="${prefix}${drive_pos}steering_link"/>
       <axis xyz="0 0 1"/>
-      <limit lower="-1" upper="1" effort="100.0" velocity="0.0"/>
+      <limit lower="-${PI}" upper="${PI}" effort="100.0" velocity="100.0"/>
       <dynamics damping="0.2"/>
-      <mimic joint="${prefix}${steering_pos}_steering_joint" multiplier="1.0" offset="${steering_mimic_offset}"/>
     </joint>
     <link name="${prefix}${drive_pos}chassis_2_link">

File: src/mobile_robot/description_mobile/urdf/mech/stand.urdf.xacro (robot description, xacro)
@@ -1,13 +1,13 @@
 <?xml version="1.0"?>
-<robot xmlns:xacro="http://wiki.ros.org/xacro">
-    <xacro:macro name="chassis" params="
+<robot xmlns:xacro="http://www.ros.org/wiki/xacro">
+    <xacro:macro name="stand" params="
         prefix parent
-        pos_z"
+        base_height"
     >
-     <link name="${prefix}chassis_link">
+     <link name="${prefix}stand_link">
         <collision>
             <origin xyz="0 0 0" rpy="0 0 0"/>
             <geometry>
-                <box size="${base_length} ${base_width} ${base_height}"/>
+                <box size="${stand_length} ${stand_width} ${stand_height}"/>
             </geometry>
         </collision>
@@ -15,7 +15,7 @@
             <origin xyz="0 0 0" rpy="0 0 0"/>
             <geometry>
-                <box size="${base_length} ${base_width} ${base_height}"/>
+                <box size="${stand_length} ${stand_width} ${stand_height}"/>
             </geometry>
-            <material name="transparent"/>
+            <material name="PETG_orange"/>
         </visual>
         <inertial>
@@ -28,8 +28,8 @@
             </inertial>
      </link>
-     <joint name="${prefix}chassis_joint" type="fixed">
+     <joint name="${prefix}stand_joint" type="fixed">
         <parent link="${prefix}${parent}"/>
-        <child link="${prefix}chassis_link"/>
-        <origin xyz="0 0 ${pos_z}" rpy="0 0 0"/>
+        <child link="${prefix}stand_link"/>
+        <origin xyz="0 0 ${str(base_height/2 + 0.20)}" rpy="0 0 0"/>
         <axis xyz="0 0 1"/>
         <dynamics damping="0.2"/>

File: src/mobile_robot/description_mobile/urdf/mech/virtual_swerve_module.urdf.xacro (robot description, xacro)
@@ -14,5 +14,5 @@
       <origin xyz="${pos_x} -${pos_y} ${pos_z}" rpy="0 0 0"/>
       <axis xyz="0 0 1"/>
-      <limit lower="-${PI}" upper="${PI}" effort="100.0" velocity="10.0"/>
+      <limit lower="-${PI}" upper="${PI}" effort="100.0" velocity="100.0"/>
     </joint>
     <!-- virtual rear left steering -->
@@ -24,5 +24,5 @@
       <origin xyz="-${pos_x} ${pos_y} ${pos_z}" rpy="0 0 0"/>
       <axis xyz="0 0 1"/>
-      <limit lower="-${PI}" upper="${PI}" effort="100.0" velocity="10.0"/>
+      <limit lower="-${PI}" upper="${PI}" effort="100.0" velocity="100.0"/>
     </joint>
     <!-- virtual rear right steering -->
@@ -34,5 +34,5 @@
       <origin xyz="-${pos_x} -${pos_y} ${pos_z}" rpy="0 0 0"/>
       <axis xyz="0 0 1"/>
-      <limit lower="-${PI}" upper="${PI}" effort="100.0" velocity="10.0"/>
+      <limit lower="-${PI}" upper="${PI}" effort="100.0" velocity="100.0"/>
     </joint>
     <!-- virtual front left steering -->
@@ -44,5 +44,5 @@
       <origin xyz="${pos_x} ${pos_y} ${pos_z}" rpy="0 0 0"/>
       <axis xyz="0 0 1"/>
-      <limit lower="-${PI}" upper="${PI}" effort="100.0" velocity="10.0"/>
+      <limit lower="-${PI}" upper="${PI}" effort="100.0" velocity="100.0"/>
     </joint>
     <!--********************************************* TRACTION *****************************************************************   -->

File: src/mobile_robot/description_mobile/urdf/properties/properties_swerveBOT_510.urdf.xacro (robot description, xacro)
@@ -6,4 +6,7 @@
   <xacro:property name="base_height" value="0.04" />
   <xacro:property name="base_mass" value="5" />
+  <xacro:property name="stand_length" value="0.400" />
+  <xacro:property name="stand_width" value="0.400" />
+  <xacro:property name="stand_height" value="0.400" />
   <xacro:property name="wheel_radius" value="0.0825" />
   <xacro:property name="wheel_len" value="0.045" />

File: src/mobile_robot/description_mobile/urdf/robots/swerve_2bot_serial.urdf.xacro (robot description, xacro)
@@ -8,4 +8,6 @@
   <xacro:arg name="command_timeout_ms" default="500"/>
   <xacro:arg name="active_modules" default="FR,RL"/>
+  <xacro:arg name="imu_topic" default="/imu/data"/>
+  <xacro:arg name="imu_frame_id" default="imu_link"/>
   <xacro:include filename="$(find description_mobile)/urdf/robots/swerve_2bot_serial_macro.xacro"/>
   <xacro:arg name="position_Z" default="${str(2*wheel_radius + base_height/2 + rulment_axial_height)}"/>
@@ -18,4 +20,6 @@
     command_timeout_ms="$(arg command_timeout_ms)"
     active_modules="$(arg active_modules)"
+    imu_topic="$(arg imu_topic)"
+    imu_frame_id="$(arg imu_frame_id)"
   />
 </robot>

File: src/mobile_robot/description_mobile/urdf/robots/swerve_2bot_serial_macro.xacro (robot description, xacro)
@@ -5,7 +5,9 @@
   <xacro:include filename="$(find description_mobile)/urdf/properties/properties_swerveBOT_510.urdf.xacro"/>
   <xacro:include filename="$(find description_mobile)/urdf/mech/chassis.urdf.xacro"/>
+  <xacro:include filename="$(find description_mobile)/urdf/mech/stand.urdf.xacro"/>
   <xacro:include filename="$(find description_mobile)/urdf/mech/serial_diff_drive_module.urdf.xacro"/>
   <xacro:include filename="$(find description_mobile)/urdf/mech/virtual_swerve_module.urdf.xacro"/>
   <xacro:include filename="$(find description_mobile)/urdf/mech/rear_wheels.urdf.xacro"/>
+  <xacro:include filename="$(find description_mobile)/urdf/sensors/imu.urdf.xacro"/>
   <xacro:include filename="$(find description_mobile)/ros2_control/wheelbot_serial_swerve_2bot.ros2_control.xacro"/>
   <xacro:macro name="wheelbot_serial_mobile_robot" params="
@@ -16,6 +18,8 @@
       baudrate
       command_timeout_ms
-      active_modules">
-    <link name="base_footprint"/>
+      active_modules
+      imu_topic
+      imu_frame_id">
+    <link name="${prefix}base_footprint"/>
     <xacro:chassis
       prefix="${prefix}"
@@ -23,7 +27,17 @@
       pos_z="${str(2*wheel_radius + base_height/2 + rulment_axial_height)}"
     />
+    <!--
+    <xacro:stand
+      prefix="${prefix}"
+      parent="chassis_link"
+      base_height="${base_height}"
+    />
+    -->
+    <xacro:imu prefix="${prefix}" parent="chassis_link" joint_name="imu_to_chassis_link">
+      <origin xyz="${wheelbase/2 - 0.05 }  0 0.26" rpy="1.57 1.57 1.57"/>
+    </xacro:imu>
     <xacro:virtual_swerve_module
       prefix="${prefix}"
-      parent="chassis_link"
+      parent="${prefix}chassis_link"
       pos_x="${str(wheelbase/2)}"
       pos_y="${str(wheel_track/2)}"
@@ -34,5 +48,5 @@
       prefix="${prefix}"
       name="diffBOT_FR"
-      parent="chassis_link"
+      parent="${prefix}chassis_link"
       drive_pos="FR_"
       steering_pos="virtual_front_right">
@@ -43,5 +57,5 @@
       prefix="${prefix}"
       name="diffBOT_RL"
-      parent="chassis_link"
+      parent="${prefix}chassis_link"
       drive_pos="RL_"
       steering_pos="virtual_rear_left"
@@ -58,4 +72,6 @@
       wheel_radius="${wheel_radius}"
       wheel_drive_len="0.23"
+      imu_topic="${imu_topic}"
+      imu_frame_id="${imu_frame_id}"
     />
   </xacro:macro>

File: src/mobile_robot/description_mobile/urdf/sensors/imu.urdf.xacro (robot description, xacro)
@@ -1,8 +1,8 @@
 <robot xmlns:xacro="http://ros.org/wiki/xacro">
-  <xacro:macro name="imu" params="*origin">
-    <link name="imu_link"/>
-    <joint name="imu_to_base_link" type="fixed">
-      <parent link="base_link"/>
-      <child link="imu_link"/>
+  <xacro:macro name="imu" params="prefix:='' parent:=base_link joint_name:=imu_to_base_link *origin">
+    <link name="${prefix}imu_link"/>
+    <joint name="${prefix}${joint_name}" type="fixed">
+      <parent link="${prefix}${parent}"/>
+      <child link="${prefix}imu_link"/>
       <xacro:insert_block name="origin" />
     </joint>
