Commit message: Use native RViz IMU display

File: src/mobile_robot/description_mobile/urdf/robots/swerve_2bot_serial_macro.xacro (robot description, xacro)
@@ -36,5 +36,5 @@
     -->
     <xacro:imu prefix="${prefix}" parent="chassis_link" joint_name="imu_to_chassis_link">
-      <origin xyz="${wheelbase/2 - 0.05 }  0 0.26" rpy="1.57 1.57 1.57"/>
+      <origin xyz="${wheelbase/2 - 0.05 }  0 0.26" rpy="1.57 0 1.57"/>
     </xacro:imu>
     <xacro:lidar.slamtec_rplidar

Commit message: Keep verified chassis IMU orientation

File: src/mobile_robot/description_mobile/urdf/robots/swerve_2bot_serial_macro.xacro (robot description, xacro)
@@ -36,5 +36,5 @@
     -->
     <xacro:imu prefix="${prefix}" parent="chassis_link" joint_name="imu_to_chassis_link">
-      <origin xyz="${wheelbase/2 - 0.05 }  0 0.26" rpy="1.57 0 1.57"/>
+      <origin xyz="${wheelbase/2 - 0.05 }  0 0.26" rpy="1.57 1.57 1.57"/>
     </xacro:imu>
     <xacro:lidar.slamtec_rplidar

Commit message: Add chassis IMU fusion and rotation validation

File: src/mobile_robot/description_mobile/urdf/robots/swerve_2bot_serial_macro.xacro (robot description, xacro)
@@ -36,5 +36,5 @@
     -->
     <xacro:imu prefix="${prefix}" parent="chassis_link" joint_name="imu_to_chassis_link">
-      <origin xyz="${wheelbase/2 - 0.05 }  0 0.26" rpy="1.57 1.57 1.57"/>
+      <origin xyz="${wheelbase/2 - 0.05 }  0 0.26" rpy="0 0 0"/>
     </xacro:imu>
     <xacro:lidar.slamtec_rplidar
